File: sch/rgb_ctrl_board/rgb_ctrl_board/rgb_ctrl_board.kicad_pcb (KiCad board)
At the start: 2 copper layers, 37 x 26 mm, 34 parts, among them J1 Conn_01x20_Male, J2 USB_B_Mini, J3 Conn_ARM_JTAG_SWD_10, U1 TLV1117-33, U2 STM32F030K6Tx, U3 FT230XS, Y1 8MHz

Commit message: skończony routing ctrl
Parts:
- removed R3, R4: 270, Resistor_SMD:R_0603_1608Metric_Pad0.98x0.95mm_HandSolder
- removed Rx1, Tx1: LED, LED_SMD:LED_0603_1608Metric_Pad1.05x0.95mm_HandSolder
- added R10: 10k, Resistor_SMD:R_0603_1608Metric_Pad0.98x0.95mm_HandSolder, F.Cu at (120.7, 129.8)
- added R9: 10k, Resistor_SMD:R_0603_1608Metric_Pad0.98x0.95mm_HandSolder, F.Cu at (120.7, 128.3)
- moved R2 4.07 mm to (120.7, 126.8)
- moved C16 2.50 mm to (125.5, 125.3)
- moved Y1 2.50 mm to (121.9, 125.2)
- moved C15 2.25 mm to (118.4, 124.9)
Connections:
- U3 pad 14: Net-(R3-Pad2) -> (no net)
- U3 pad 7: Net-(R4-Pad2) -> (no net)
Routing:
- net Net-(R2-Pad2): track 0.00 -> 21.1 mm, vias 0 -> 2
- net Net-(C1-Pad1): track 11.5 -> 29.2 mm, vias 2 -> 4
- net Net-(C16-Pad1): track 0.00 -> 6.89 mm, vias 0 -> 1
- net Net-(C15-Pad1): track 1.72 -> 8.17 mm, vias 0 -> 1
- net +3V3: track 94.2 -> 99.1 mm, vias 3 -> 5
- net /RESET: track 33.6 -> 36.2 mm
- net /USART1_Rx: track 10.1 -> 7.63 mm
- net Net-(R10-Pad1): track 11.2 -> 10.1 mm
- net (no net): vias 0 -> 1

Commit message: drobne poprawki
Parts:
- moved Y1 0.50 mm to (121.9, 125.7)
- moved C16 0.20 mm to (125.7, 125.3)
- moved C15 0.10 mm to (118.3, 124.9)
Routing:
- net GND: track 18.8 -> 16.1 mm, vias 29 -> 34
- net Net-(C14-Pad1): track 17.6 -> 20.1 mm
- net LED4: track 18.9 -> 21.3 mm
- net LED2: track 16.6 -> 18.1 mm
- net Net-(C15-Pad1): track 8.17 -> 9.58 mm
- net Net-(C16-Pad1): track 6.89 -> 8.15 mm
- net +3V3: track 99.1 -> 100.0 mm
- net (no net): vias 1 -> 0

Commit message: add gerber files
Changed lines of the file:
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@@
   (general
     (thickness 1.6)
-    (drawings 4)
+    (drawings 6)
     (tracks 414)
     (zones 0)
@@
     (38 B.Mask user hide)
     (39 F.Mask user hide)
-    (40 Dwgs.User user hide)
-    (41 Cmts.User user hide)
+    (40 Dwgs.User user)
+    (41 Cmts.User user)
     (42 Eco1.User user hide)
     (43 Eco2.User user hide)
@@
     (visible_elements 7FFFFFFF)
     (pcbplotparams
-      (layerselection 0x010fc_ffffffff)
+      (layerselection 0x010f0_ffffffff)
       (usegerberextensions false)
       (usegerberattributes true)
@@
       (outputformat 1)
       (mirror false)
-      (drillshape 1)
+      (drillshape 0)
       (scaleselection 1)
-      (outputdirectory ""))
+      (outputdirectory "gerber"))
   )
   (net 0 "")
@@
     (pad 3 thru_hole circle (at 2 0 270) (size 1.2 1.2) (drill 0.75) (layers *.Cu *.Mask)
       (net 1 GND))
-    (pad 1 thru_hole roundrect (at 0 0 270) (size 1.2 1.2) (drill 0.75) (layers *.Cu *.Mask) (roundrect_rratio 0.208333)
+    (pad 1 thru_hole roundrect (at 0 0 270) (size 1.2 1.2) (drill 0.75) (layers *.Cu *.Mask) (roundrect_rratio 0.2083325)
       (net 3 +3V3))
     (model ${KISYS3DMOD}/Connector_JST.3dshapes/JST_PHD_S20B-PHDSS_2x10_P2.00mm_Horizontal.wrl
@@
     )
   )
+  (dimension 26 (width 0.12) (layer Dwgs.User)
+    (gr_text "26,000 mm" (at 150.94 120 90) (layer Dwgs.User)
+      (effects (font (size 0.7 0.7) (thickness 0.12)))
+    )
+    (feature1 (pts (xy 148 107) (xy 150.586421 107)))
+    (feature2 (pts (xy 148 133) (xy 150.586421 133)))
+    (crossbar (pts (xy 150 133) (xy 150 107)))
+    (arrow1a (pts (xy 150 107) (xy 150.586421 108.126504)))
+    (arrow1b (pts (xy 150 107) (xy 149.413579 108.126504)))
+    (arrow2a (pts (xy 150 133) (xy 150.586421 131.873496)))
+    (arrow2b (pts (xy 150 133) (xy 149.413579 131.873496)))
+  )
+  (dimension 37 (width 0.12) (layer Dwgs.User)
+    (gr_text "37,000 mm" (at 129.5 135.94) (layer Dwgs.User)
+      (effects (font (size 0.7 0.7) (thickness 0.12)))
+    )
+    (feature1 (pts (xy 148 133) (xy 148 135.586421)))
+    (feature2 (pts (xy 111 133) (xy 111 135.586421)))
+    (crossbar (pts (xy 111 135) (xy 148 135)))
+    (arrow1a (pts (xy 148 135) (xy 146.873496 135.586421)))
+    (arrow1b (pts (xy 148 135) (xy 146.873496 134.413579)))
+    (arrow2a (pts (xy 111 135) (xy 112.126504 135.586421)))
+    (arrow2b (pts (xy 111 135) (xy 112.126504 134.413579)))
+  )
   (gr_line (start 148 133) (end 148 107) (layer Edge.Cuts) (width 0.05))
